Commit message: Latest dev

File: copernicus_description/urdf/vehicle_properties.xacro (robot description, xacro)
@@ -85,12 +85,15 @@
     <xacro:property name="velodyne_mount_iyz" value="0.000"/>
     <xacro:property name="velodyne_mount_izz" value="0.002"/>
-    <xacro:property name="velodyne_mount_joint_x" value="0.259"/>
+    <!-- <xacro:property name="velodyne_mount_joint_x" value="0.259"/> -->
+    <xacro:property name="velodyne_mount_joint_x" value="-0.027"/>
     <xacro:property name="velodyne_mount_joint_y" value="-0.0625"/>
-    <xacro:property name="velodyne_mount_joint_z" value="0.296"/>
-    <xacro:property name="velodyne_mount_joint_pitch" value="0.415"/>
+    <xacro:property name="velodyne_mount_joint_z" value="0.30"/>
+    <!-- <xacro:property name="velodyne_mount_joint_pitch" value="0.415"/> -->
+    <xacro:property name="velodyne_mount_joint_pitch" value="0.0"/>
     <xacro:property name="velodyne_joint_x" value="0.027"/>
     <xacro:property name="velodyne_joint_y" value="0.0625"/>
     <xacro:property name="velodyne_joint_z" value="0.0295"/>
-    <xacro:property name="velodyne_joint_pitch" value="0.262"/>
+    <!-- <xacro:property name="velodyne_joint_pitch" value="0.262"/> -->
+    <xacro:property name="velodyne_joint_pitch" value="0.0"/>
     <xacro:property name="dummy_inertia" value="1e-09"/>
     <xacro:property name="dummy_inertia" value="1e-09"/>
