Commit message: Latest development

File: copernicus_description/urdf/copernicus.urdf.xacro (robot description, xacro)
@@ -102,5 +102,5 @@
             <xacro:include filename="$(find velodyne_description)/urdf/VLP-16.urdf.xacro"/>
             <VLP-16 parent="velodyne_mount" name="velodyne" topic="velodyne_points" hz="10" samples="440" gpu="false" min_range="0.2">
-                <origin xyz="${velodyne_joint_x} ${velodyne_joint_y} ${velodyne_joint_z}" rpy="0 ${-velodyne_joint_pitch} 0" />
+                <origin xyz="${velodyne_joint_x} ${velodyne_joint_y} ${velodyne_joint_z}" rpy="${velodyne_joint_roll} ${-velodyne_joint_pitch} ${velodyne_joint_yaw}" />
             </VLP-16>
         </xacro:if>

File: copernicus_description/urdf/vehicle_properties.xacro (robot description, xacro)
@@ -86,7 +86,7 @@
     <xacro:property name="velodyne_mount_izz" value="0.002"/>
     <!-- <xacro:property name="velodyne_mount_joint_x" value="0.259"/> -->
-    <xacro:property name="velodyne_mount_joint_x" value="-0.027"/>
+    <xacro:property name="velodyne_mount_joint_x" value="-0.177"/>
     <xacro:property name="velodyne_mount_joint_y" value="-0.0625"/>
-    <xacro:property name="velodyne_mount_joint_z" value="0.30"/>
+    <xacro:property name="velodyne_mount_joint_z" value="0.43"/>
     <!-- <xacro:property name="velodyne_mount_joint_pitch" value="0.415"/> -->
     <xacro:property name="velodyne_mount_joint_pitch" value="0.0"/>
@@ -95,5 +95,7 @@
     <xacro:property name="velodyne_joint_z" value="0.0295"/>
     <!-- <xacro:property name="velodyne_joint_pitch" value="0.262"/> -->
+    <xacro:property name="velodyne_joint_roll" value="0.0"/>
     <xacro:property name="velodyne_joint_pitch" value="0.0"/>
+    <xacro:property name="velodyne_joint_yaw" value="3.14"/>
     <xacro:property name="dummy_inertia" value="1e-09"/>
     <xacro:property name="dummy_inertia" value="1e-09"/>
